File: PCB/EAGLE/PCB.sch (EAGLE design)
At the start: 82 parts, among them SW1 EC12E_SW

Commit message: D_groups
Parts:
- added D10, D11, D12, D13, D14, D15, D16, D17, D18, D19, D2, D20, D21, D22, D23, D24, D25, D26, D27, D28, D29, D3, D30, D31, D32, D33, D34, D35, D36, D37, D38, D39, D4, D40, D41, D42, D43, D44, D45, D46, D47, D48, D49, D5, D50, D51, D52, D53, D54, D55, D56, D57, D58, D59, D6, D60, D61, D62, D63, D64, D65, D66, D67, D68, D69, D7, D70, D71, D72, D73, D74, D75, D76, D8, D9: (no value), Components:DIODE-SOD-123
Connections:
- new net N$1: D2.A, ESC.P0
- new net N$10: D10.A, F9.P0
- new net N$11: D11.A, F10.P0
- new net N$12: D12.A, F11.P0
- new net N$13: D13.A, F12.P0
- new net N$14: D14.A, ~.P0
- new net N$15: 1.P0, D15.A
- new net N$16: 2.P0, D16.A
- new net N$17: 3.P0, D17.A
- new net N$18: 4.P0, D18.A
- new net N$19: 5.P0, D19.A
- new net N$2: D1.A, F1.P0
- new net N$20: 6.P0, D20.A
- new net N$21: 7.P0, D21.A
- new net N$22: 8.P0, D22.A
- new net N$23: 9.P0, D23.A
- new net N$24: 0.P0, D24.A
- new net N$25: -.P0, D25.A
- new net N$26: +.P0, D26.A
- new net N$27: D27.A, DELETE.P0
- new net N$28: D28.A, PAGEUP.P0
- new net N$29: D29.A, PAGEDOWN.P0
- new net N$3: D3.A, F2.P0
- new net N$30: D30.A, Q.P0
- new net N$31: D31.A, W.P0
- new net N$32: D32.A, E.P0
- new net N$33: D33.A, R.P0
- new net N$34: D34.A, T.P0
- new net N$35: D35.A, Y.P0
- new net N$36: D36.A, U.P0
- new net N$37: D37.A, I.P0
- new net N$38: D38.A, O.P0
- new net N$39: D39.A, P.P0
- new net N$4: D4.A, F3.P0
- new net N$40: D40.A, [.P0
- new net N$41: D41.A, ].P0
- new net N$42: BACKSLASH.P0, D42.A
- new net N$43: A.P0, D43.A
- new net N$44: D44.A, S.P0
- new net N$45: D.P0, D45.A
- new net N$46: D46.A, F.P0
- new net N$47: D47.A, G.P0
- new net N$48: D48.A, H.P0
- new net N$49: D49.A, J.P0
- new net N$5: D5.A, F4.P0
- new net N$50: D50.A, K.P0
- new net N$51: D51.A, L.P0
- new net N$52: D52.A, DOUBLEDOTS.P0
- new net N$53: D53.A, TOPAND.P0
- new net N$54: D54.A, Z.P0
- new net N$55: D55.A, X.P0
- new net N$56: C.P0, D56.A
- new net N$57: D57.A, V.P0
- new net N$58: B.P0, D58.A
- new net N$59: D59.A, N.P0
- new net N$6: D6.A, F5.P0
- new net N$60: D60.A, M.P0
- new net N$61: BOTTOMAND.P0, D61.A
- new net N$62: D62.A, DOT.P0
- new net N$63: ASKW.P0, D63.A
- new net N$64: D64.A, LCTRL.P0
- new net N$65: D65.A, WIN.P0
- new net N$66: D66.A, LALT.P0
- new net N$67: D67.A, SPACE.P0
- new net N$68: D68.A, RALT.P0
- new net N$69: D69.A, RCTRL.P0
- new net N$7: D7.A, F6.P0
- new net N$70: D70.A, FN.P0
- new net N$71: D71.A, LEFT.P0
- new net N$72: D72.A, UP.P0
- new net N$73: D73.A, DOWN.P0
- new net N$74: D74.A, RIGHT.P0
- new net N$75: D75.A, TAB.P0
- new net N$76: CAPS.P0, D76.A
- new net N$8: D8.A, F7.P0
- new net N$9: D9.A, F8.P0
Other:
- moved on the sheet: D1
